Commit message: success on ussing joystick

File: description/camera.xacro (robot description, xacro)
@@ -1,13 +1,13 @@
 <?xml version="1.0"?>
 <robot xmlns:xacro="http://www.ros.org/wiki/xacro" >
-    <joint name="camera_joint" type="fixed">
+    <!-- <joint name="camera_joint" type="fixed">
         <parent link="chassis"/>
         <child link="camera_link"/>
-        <origin xyz="0.305 0 0.08" rpy="0 0 0"/>
+        <origin xyz="0.224 0 0.098" rpy="0 0 0"/>
     </joint>
     <link name="camera_link">
         <visual>
             <geometry>
-                <box size="0.010 0.03 0.03"/>
+                <box size="0.108 0.045 0.045"/>
             </geometry>
             <material name="red"/>
@@ -42,4 +42,4 @@
             </plugin>
         </sensor>
-    </gazebo>
+    </gazebo> -->
 </robot>

File: description/gazebo_control.xacro (robot description, xacro)
@@ -21,4 +21,9 @@
             <publish_wheel_tf>true</publish_wheel_tf>
         </plugin>
+        <!-- Camera Joint Plugin -->
+        <plugin name='camera_joint_controller' filename='libgazebo_ros_control.so'>
+            <camera_joint>camera_joint</camera_joint>
+            <pid>1.0 0.0 0.0</pid>
+        </plugin>
     </gazebo>
 </robot>

File: description/robot_core.xacro (robot description, xacro)
@@ -152,3 +152,29 @@
         <mu2 value="0.001"/>
     </gazebo>
+    <!-- //////////////////////////////////////////////////////////////////// -->
+    <joint name="camera_joint" type="continuous">
+        <parent link="chassis"/>
+        <child link="camera_link"/>
+        <origin xyz="0.224 0 0.098" rpy="0 0 0"/>
+        <axis xyz="0 0 1"/>
+    </joint>
+    <link name="camera_link">
+        <visual>
+            <geometry>
+                <box size="0.108 0.045 0.045"/>
+            </geometry>
+            <material name="red"/>
+        </visual>
+        <collision>
+            <geometry>
+                <box size="0.108 0.045 0.045"/>
+            </geometry>
+        </collision>
+        <xacro:inertial_box mass="0.5" x="0.108" y="0.045" z="0.045">
+            <origin xyz="0 0 0" rpy="0 0 0"/>
+        </xacro:inertial_box>
+    </link>
+    <gazebo reference="camera_link">
+        <material>Gazebo/Red</material>
+    </gazebo>
 </robot>

File: description/ros2_control.xacro (robot description, xacro)
@@ -21,4 +21,13 @@
             <state_interface name="position"/>
         </joint>
+        <!-- /////////////////////////////////////////////////////////////////////// -->
+        <joint name="camera_joint">
+            <command_interface name="velocity">
+                <param name="min">-10</param>
+                <param name="max">10</param>
+            </command_interface>
+            <state_interface name="velocity"/>
+            <state_interface name="position"/>
+        </joint>
     </ros2_control>
     <gazebo>
